File: MurataSD.brd (EAGLE design)
At the start: 50 x 52 mm, 0 parts

Commit message: [ NEW ] BOARD_MMC
Parts:
- added U1: IC_BLE_LBCA2HNZYZ-711, mylib:IC_MURATA_LBCA2HNZYZ-711
- added U100: BOARD_MMC, mylib:BOARD_MMC
Other:
- outline, holes or cut-outs redrawn
