File: MurataSD.sch (EAGLE design)
At the start: 0 parts

Commit message: [ NEW ] BOARD_MMC
Parts:
- added U1: IC_BLE_LBCA2HNZYZ-711, mylib:IC_BLE_LBCA2HNZYZ-711
- added U100: BOARD_MMC, mylib:BOARD_MMC
