File: MurataMicroSD.brd (EAGLE design)
At the start: 25.6 x 12.8 mm, 9 parts, among them U1 IC_BLE_LBCA2HNZYZ-711

Commit message: [ FIX ] MurataMicroSD
add via for GND
Routing:
- net GND: vias 12 -> 21
Changed lines of the file:
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@@
 <via x="4.7" y="9.5" extent="1-16" drill="0.3"/>
 <wire x1="2.4" y1="9.5" x2="4.7" y2="9.5" width="0.8" layer="16"/>
+<via x="20.6" y="15.3" extent="1-16" drill="0.3"/>
+<via x="20.1" y="14.8" extent="1-16" drill="0.3"/>
+<via x="20.6" y="14.3" extent="1-16" drill="0.3"/>
+<via x="19.6" y="12.6" extent="1-16" drill="0.3"/>
+<via x="20.6" y="13" extent="1-16" drill="0.3"/>
+<via x="20.6" y="6.7" extent="1-16" drill="0.3"/>
+<via x="20.1" y="6.2" extent="1-16" drill="0.3"/>
+<via x="20.6" y="5.7" extent="1-16" drill="0.3"/>
+<via x="19.6" y="8.4" extent="1-16" drill="0.3"/>
 </signal>
 <signal name="N$1">

Commit message: [ FIX ] SCH change; library update myPCBlib: 385519d7d8f28a1be9991780ecc3cf499a6be8e2
Parts:
- added TP6, TP7, TP8: TPTP08R, testpad_local:TP08R
- moved TP1 0.10 mm to (15.6, 6.00)
Connections:
- removed net N$8: U1.11
- removed net TXD_MISO: C100.7_MISO, U1.2
- new net MISO: C100.7_MISO, U1.23
- new net N$2: TP6.TP, U1.31
- new net P0_2: TP8.TP, U1.12
- new net P0_3: TP7.TP, U1.11
- net !CS!: now also U1.2; no longer U1.23
- net DAT1: now also U1.22; no longer U1.3
- net DAT2: now also U1.3; no longer U1.22
Routing:
- net MISO: track 0.00 -> 17.6 mm
- net TXD_MISO: track 16.1 -> 0.00 mm, vias 1 -> 0
- net N$2: track 0.00 -> 3.25 mm, vias 0 -> 1
- net P0_3: track 0.00 -> 1.99 mm
- net DAT2: track 18.0 -> 16.2 mm, vias 1 -> 0
- net DAT1: track 16.2 -> 18.0 mm, vias 1 -> 0
- net P0_2: track 0.00 -> 1.74 mm
- net !CS!: track 17.6 -> 16.1 mm, vias 1 -> 0
- net RXD_MOSI: track 17.1 -> 18.4 mm, vias 1 -> 0
- net GND: track 4.60 -> 4.10 mm
- net SCK: track 17.1 -> 16.6 mm, vias 3 -> 2
- net 3.3V: track 16.6 -> 16.1 mm, vias 1 -> 2

Commit message: [ FIX ] library update; trace; increase via myPCBlib: 0aa2107fd28665ba7552473a3fbc4a367f8d93bf
Routing:
- net GND: vias 21 -> 23
Changed lines of the file:
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@@
 <wire x1="2.4" y1="10.6" x2="4.9" y2="10.6" width="0.8" layer="1"/>
 <via x="4.9" y="10.6" extent="1-16" drill="0.3"/>
+<wire x1="17.2" y1="8.55" x2="17.1" y2="8.55" width="0" layer="19" extent="1-1"/>
 </signal>
 <signal name="GND">
@@
 <vertex x="0" y="5"/>
 </polygon>
-<via x="17.9" y="9.1" extent="1-16" drill="0.3"/>
-<via x="18" y="10" extent="1-16" drill="0.3"/>
-<via x="18" y="11" extent="1-16" drill="0.3"/>
+<via x="17.8" y="9.2" extent="1-16" drill="0.3"/>
+<via x="18.7" y="10" extent="1-16" drill="0.3"/>
+<via x="18.7" y="11" extent="1-16" drill="0.3"/>
 <polygon width="0.25" layer="1" thermals="no">
 <vertex x="15" y="16"/>
@@
 <wire x1="15.7" y1="7.4" x2="15.2" y2="7.4" width="0.6" layer="1"/>
 <wire x1="15.2" y1="7.4" x2="14.9" y2="7.4" width="0.8" layer="1"/>
-<via x="18.4" y="12" extent="1-16" drill="0.3"/>
-<via x="19.6" y="11.9" extent="1-16" drill="0.3"/>
-<via x="19.6" y="11" extent="1-16" drill="0.3"/>
-<via x="19.6" y="10.1" extent="1-16" drill="0.3"/>
-<via x="19.6" y="9.2" extent="1-16" drill="0.3"/>
+<via x="17.9" y="11.7" extent="1-16" drill="0.3"/>
+<via x="19.5" y="11.9" extent="1-16" drill="0.3"/>
+<via x="19.5" y="11" extent="1-16" drill="0.3"/>
+<via x="19.5" y="10" extent="1-16" drill="0.3"/>
+<via x="19.6" y="9.3" extent="1-16" drill="0.3"/>
 <contactref element="R1" pad="1"/>
 <via x="14.9" y="12.3" extent="1-16" drill="0.3"/>
@@
 <via x="20.1" y="14.8" extent="1-16" drill="0.3"/>
 <via x="20.6" y="14.3" extent="1-16" drill="0.3"/>
-<via x="19.6" y="12.6" extent="1-16" drill="0.3"/>
-<via x="20.6" y="13" extent="1-16" drill="0.3"/>
+<via x="19.7" y="12.6" extent="1-16" drill="0.3"/>
+<via x="20.6" y="12.9" extent="1-16" drill="0.3"/>
 <via x="20.6" y="6.7" extent="1-16" drill="0.3"/>
 <via x="20.1" y="6.2" extent="1-16" drill="0.3"/>
@@
 <wire x1="2.4" y1="12.8" x2="4.9" y2="12.8" width="0.8" layer="1"/>
 <via x="16.8" y="7.3" extent="1-16" drill="0.3"/>
+<via x="17.9" y="11" extent="1-16" drill="0.3"/>
+<via x="17.9" y="10" extent="1-16" drill="0.3"/>
 </signal>
 <signal name="N$1">
 <contactref element="U1" pad="25"/>
 <contactref element="R1" pad="2"/>
-<wire x1="17.75" y1="13.4" x2="17.75" y2="13.75" width="0.25" layer="1"/>
-<wire x1="17.75" y1="13.75" x2="17.5" y2="14" width="0.25" layer="1"/>
-<wire x1="17.5" y1="14" x2="16.2" y2="14" width="0.25" layer="1"/>
 <wire x1="16.2" y1="14" x2="15.7" y2="13.5" width="0.25" layer="1"/>
+<wire x1="17.725" y1="13.4" x2="17.725" y2="13.875" width="0.25" layer="1"/>
+<wire x1="17.725" y1="13.875" x2="17.6" y2="14" width="0.25" layer="1"/>
+<wire x1="17.6" y1="14" x2="16.2" y2="14" width="0.25" layer="1"/>
 </signal>
 <signal name="MISO">
 <contactref element="U1" pad="23"/>
-<wire x1="18.95" y1="13.4" x2="18.95" y2="13.75" width="0.25" layer="1"/>
-<wire x1="18.95" y1="13.75" x2="17.9" y2="14.8" width="0.25" layer="1"/>
-<wire x1="17.9" y1="14.8" x2="15" y2="14.8" width="0.25" layer="1"/>
+<wire x1="18.4" y1="14.8" x2="15" y2="14.8" width="0.25" layer="1"/>
 <wire x1="15" y1="14.8" x2="14.1" y2="13.9" width="0.25" layer="1"/>
 <wire x1="4.1" y1="13.9" x2="14.1" y2="13.9" width="0.25" layer="1"/>
 <contactref element="C100" pad="7_MISO"/>
 <wire x1="2.55" y1="13.9" x2="4.1" y2="13.9" width="0.8" layer="1"/>
+<wire x1="19.025" y1="13.4" x2="19.025" y2="14.175" width="0.25" layer="1"/>
+<wire x1="19.025" y1="14.175" x2="18.4" y2="14.8" width="0.25" layer="1"/>
 </signal>
 <signal name="DAT1">
 <contactref element="U1" pad="22"/>
-<wire x1="19.55" y1="13.4" x2="19.55" y2="13.75" width="0.25" layer="1"/>
-<wire x1="19.55" y1="13.75" x2="18.1" y2="15.2" width="0.25" layer="1"/>
-<wire x1="18.1" y1="15.2" x2="14.5" y2="15.2" width="0.25" layer="1"/>
+<wire x1="18.7" y1="15.2" x2="14.5" y2="15.2" width="0.25" layer="1"/>
 <wire x1="14.5" y1="15.2" x2="14.3" y2="15" width="0.25" layer="1"/>
 <wire x1="4.1" y1="15" x2="14.3" y2="15" width="0.25" layer="1"/>
 <contactref element="C100" pad="8_DAT1"/>
 <wire x1="2.55" y1="15" x2="4.1" y2="15" width="0.8" layer="1"/>
+<wire x1="19.675" y1="13.4" x2="19.675" y2="14.225" width="0.25" layer="1"/>
+<wire x1="19.675" y1="14.225" x2="18.7" y2="15.2" width="0.25" layer="1"/>
 </signal>
 <signal name="RXD_MOSI">
 <contactref element="U1" pad="24"/>
-<wire x1="18.35" y1="13.4" x2="18.35" y2="13.75" width="0.25" layer="1"/>
-<wire x1="18.35" y1="13.75" x2="17.7" y2="14.4" width="0.25" layer="1"/>
-<wire x1="17.7" y1="14.4" x2="15.4" y2="14.4" width="0.25" layer="1"/>
+<wire x1="18.2" y1="14.4" x2="15.4" y2="14.4" width="0.25" layer="1"/>
 <wire x1="15.4" y1="14.4" x2="13" y2="12" width="0.25" layer="1"/>
 <wire x1="13" y1="12" x2="10.5" y2="12" width="0.25" layer="1"/>
@@
 <contactref element="C100" pad="3_MOSI"/>
 <wire x1="2.55" y1="9.5" x2="4.1" y2="9.5" width="0.8" layer="1"/>
+<wire x1="18.375" y1="13.4" x2="18.375" y2="14.225" width="0.25" layer="1"/>
+<wire x1="18.375" y1="14.225" x2="18.2" y2="14.4" width="0.25" layer="1"/>
 </signal>
 <signal name="!CS!">
@@
 <contactref element="C100" pad="2_CS"/>
 <wire x1="2.55" y1="8.4" x2="4.1" y2="8.4" width="0.8" layer="1"/>
+<wire x1="17.2" y1="11.8" x2="17.1" y2="11.8" width="0" layer="19" extent="1-1"/>
 </signal>
 <signal name="DAT2">
@@
 <contactref element="C100" pad="1_DAT2"/>
 <wire x1="2.55" y1="7.3" x2="4.1" y2="7.3" width="0.8" layer="1"/>
+<wire x1="17.2" y1="11.15" x2="17.1" y2="11.15" width="0" layer="19" extent="1-1"/>
 </signal>
 <signal name="P0_3">
 <contactref element="U1" pad="11"/>
 <contactref element="TP7" pad="TP"/>
-<wire x1="18.95" y1="7.6" x2="18.95" y2="7.15" width="0.25" layer="1"/>
-<wire x1="18.95" y1="7.15" x2="18" y2="6.2" width="0.25" layer="1"/>
-<wire x1="18" y1="6" x2="18" y2="6.2" width="0.25" layer="1"/>
+<wire x1="19.025" y1="7.6" x2="19.025" y2="7.125" width="0.25" layer="1"/>
+<wire x1="19.025" y1="7.125" x2="18.8" y2="6.9" width="0.25" layer="1"/>
+<wire x1="18" y1="6" x2="18" y2="6.7" width="0.25" layer="1"/>
+<wire x1="18" y1="6.7" x2="18.2" y2="6.9" width="0.25" layer="1"/>
+<wire x1="18.2" y1="6.9" x2="18.8" y2="6.9" width="0.25" layer="1"/>
 </signal>
 <signal name="SCK">
@@
 <wire x1="2.55" y1="11.7" x2="4.1" y2="11.7" width="0.8" layer="1"/>
 <via x="12.7" y="12.9" extent="1-16" drill="0.3"/>
+<wire x1="17.2" y1="12.45" x2="17.1" y2="12.45" width="0" layer="19" extent="1-1"/>
 </signal>
 <signal name="SWCLK">
@@
 <wire x1="13.4" y1="6.3" x2="13.4" y2="9.9" width="0.25" layer="1"/>
 <wire x1="13.4" y1="9.9" x2="14" y2="10.5" width="0.25" layer="1"/>
+<wire x1="17.2" y1="10.5" x2="17.1" y2="10.5" width="0" layer="19" extent="1-1"/>
 </signal>
 <signal name="SWDIO">
@@
 <wire x1="14.1" y1="6.9" x2="14.1" y2="9.6" width="0.25" layer="1"/>
 <wire x1="14.1" y1="9.6" x2="14.5" y2="10" width="0.25" layer="1"/>
+<wire x1="17.2" y1="9.85" x2="17.1" y2="9.85" width="0" layer="19" extent="1-1"/>
 </signal>
 <signal name="N$2">
 <contactref element="TP6" pad="TP"/>
 <contactref element="U1" pad="31"/>
-<wire x1="18.975" y1="8.55" x2="19.45" y2="8.55" width="0.25" layer="1"/>
-<wire x1="19.45" y1="8.55" x2="19.6" y2="8.4" width="0.25" layer="1"/>
-<via x="19.6" y="8.4" extent="1-16" drill="0.3"/>
-<wire x1="19.2" y1="6" x2="19.2" y2="6.7" width="0.25" layer="16"/>
-<wire x1="19.2" y1="6.7" x2="19.6" y2="7.1" width="0.25" layer="16"/>
-<wire x1="19.6" y1="7.1" x2="19.6" y2="8.4" width="0.25" layer="16"/>
+<wire x1="19.025" y1="8.65" x2="19.35" y2="8.65" width="0.25" layer="1"/>
+<wire x1="19.35" y1="8.65" x2="19.5" y2="8.5" width="0.25" layer="1"/>
+<via x="19.5" y="8.5" extent="1-16" drill="0.3"/>
+<wire x1="19.5" y1="8.5" x2="19.5" y2="7.4" width="0.25" layer="16"/>
+<wire x1="19.5" y1="7.4" x2="19.2" y2="7.1" width="0.25" layer="16"/>
+<wire x1="19.2" y1="7.1" x2="19.2" y2="6" width="0.25" layer="16"/>
 </signal>
 <signal name="P0_2">
 <contactref element="TP8" pad="TP"/>
 <contactref element="U1" pad="12"/>
-<wire x1="19.55" y1="7.6" x2="19.55" y2="7.05" width="0.25" layer="1"/>
-<wire x1="19.55" y1="7.05" x2="19.2" y2="6.7" width="0.25" layer="1"/>
-<wire x1="19.2" y1="6.7" x2="19.2" y2="6" width="0.25" layer="1"/>
+<wire x1="19.2" y1="6" x2="19.2" y2="6.5" width="0.25" layer="1"/>
+<wire x1="19.2" y1="6.5" x2="19.675" y2="6.975" width="0.25" layer="1"/>
+<wire x1="19.675" y1="7.6" x2="19.675" y2="6.975" width="0.25" layer="1"/>
 </signal>
 </signals>
