File: MurataMicroSD.sch (EAGLE design)
At the start: 9 parts, among them U1 IC_BLE_LBCA2HNZYZ-711

Commit message: [ FIX ] SCH change; library update myPCBlib: 385519d7d8f28a1be9991780ecc3cf499a6be8e2
Parts:
- added TP6, TP7, TP8: TPTP08R, testpad_local:TPTP08R
Connections:
- removed net N$8: U1.P0_3
- removed net TXD_MISO: C100.7, U1.P0_7
- new net MISO: C100.7, U1.P0_0
- new net N$2: TP6.TP, U1.VPP
- new net P0_2: TP8.TP, U1.P0_2
- new net P0_3: TP7.TP, U1.P0_3
- net !CS!: now also U1.P0_7; no longer U1.P0_0
- net DAT1: now also U1.P0_1; no longer U1.P0_6
- net DAT2: now also U1.P0_6; no longer U1.P0_1
Other:
- note added: "-> P0_4/RXD/MOSI"
- note added: "<- P0_0/TXD/MISO"
- note added: "P0_0/TXD/MISO ->"
- note added: "P0_1/DAT1"
- note added: "P0_4/RXD/MOSI <-"
- note added: "P0_5/SCK"
- note added: "P0_6/DAT2"
- note added: "P0_7/!CS!"
- moved on the sheet: C1, R1, TP1, TP2, U1

Commit message: [ FIX ] BLE module placed on top
other side of uSD contacts
Connections:
- net !CS!: now also U1.P0_0; no longer U1.P0_7
- net DAT1: now also U1.P0_6; no longer U1.P0_1
- net DAT2: now also U1.P0_1; no longer U1.P0_6
- net MISO: now also U1.P0_7; no longer U1.P0_0
Other:
- note added: "<- P0_7/TXD/MISO"
- note added: "P0_0/!CS!"
- note added: "P0_1/DAT2"
- note added: "P0_6/DAT1"
- note added: "P0_7/TXD/MISO->"
- note removed: "<- P0_0/TXD/MISO"
- note removed: "P0_0/TXD/MISO ->"
- note removed: "P0_1/DAT1"
- note removed: "P0_6/DAT2"
- note removed: "P0_7/!CS!"
Changed lines of the file:
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@@
 <circle x="223.52" y="38.1" radius="12.7" width="0.1524" layer="91"/>
 <text x="218.44" y="27.94" size="1.778" layer="91">FIDUCIAL</text>
-<text x="152.4" y="111.76" size="1.778" layer="94">P0_0/TXD/MISO -&gt;</text>
-<text x="152.4" y="109.22" size="1.778" layer="94">P0_1/DAT1</text>
-<text x="152.4" y="101.6" size="1.778" layer="94">P0_4/RXD/MOSI &lt;-</text>
-<text x="152.4" y="99.06" size="1.778" layer="94">P0_5/SCK</text>
-<text x="152.4" y="96.52" size="1.778" layer="94">P0_6/DAT2</text>
-<text x="71.12" y="83.82" size="1.778" layer="94" rot="MR0">P0_6/DAT2</text>
+<text x="154.94" y="111.76" size="1.778" layer="94">P0_0/!CS!</text>
+<text x="154.94" y="109.22" size="1.778" layer="94">P0_1/DAT2</text>
+<text x="154.94" y="101.6" size="1.778" layer="94">P0_4/RXD/MOSI &lt;-</text>
+<text x="154.94" y="99.06" size="1.778" layer="94">P0_5/SCK</text>
+<text x="154.94" y="96.52" size="1.778" layer="94">P0_6/DAT1</text>
+<text x="71.12" y="83.82" size="1.778" layer="94" rot="MR0">P0_1/DAT2</text>
 <text x="71.12" y="104.14" size="1.778" layer="94" rot="MR0">P0_5/SCK</text>
 <text x="71.12" y="93.98" size="1.778" layer="94" rot="MR0">-&gt; P0_4/RXD/MOSI</text>
@@
 <wire x1="193.04" y1="76.2" x2="193.04" y2="127" width="0.254" layer="94"/>
 <wire x1="193.04" y1="127" x2="99.06" y2="127" width="0.254" layer="94"/>
-<text x="71.12" y="114.3" size="1.778" layer="94" align="bottom-right">&lt;- P0_0/TXD/MISO</text>
-<text x="71.12" y="119.38" size="1.778" layer="94" rot="MR0">P0_1/DAT1</text>
-<text x="152.4" y="93.98" size="1.778" layer="94">P0_7/!CS!</text>
-<text x="71.12" y="88.9" size="1.778" layer="94" rot="MR0">P0_7/!CS!</text>
+<text x="71.12" y="114.3" size="1.778" layer="94" align="bottom-right">&lt;- P0_7/TXD/MISO</text>
+<text x="71.12" y="119.38" size="1.778" layer="94" rot="MR0">P0_6/DAT1</text>
+<text x="154.94" y="93.98" size="1.778" layer="94">P0_7/TXD/MISO-&gt;</text>
+<text x="71.12" y="88.9" size="1.778" layer="94" rot="MR0">P0_0/!CS!</text>
 </plain>
 <instances>
@@
 <net name="MISO" class="0">
 <segment>
-<pinref part="U1" gate="G$1" pin="P0_0"/>
-<wire x1="144.78" y1="111.76" x2="152.4" y2="111.76" width="0.1524" layer="91"/>
+<wire x1="81.28" y1="114.3" x2="71.12" y2="114.3" width="0.1524" layer="91"/>
+<pinref part="C100" gate="G$1" pin="7"/>
 </segment>
 <segment>
-<wire x1="81.28" y1="114.3" x2="71.12" y2="114.3" width="0.1524" layer="91"/>
-<pinref part="C100" gate="G$1" pin="7"/>
+<wire x1="154.94" y1="93.98" x2="144.78" y2="93.98" width="0.1524" layer="91"/>
+<pinref part="U1" gate="G$1" pin="P0_7"/>
 </segment>
 </net>
 <net name="DAT1" class="0">
 <segment>
-<pinref part="U1" gate="G$1" pin="P0_1"/>
-<wire x1="144.78" y1="109.22" x2="152.4" y2="109.22" width="0.1524" layer="91"/>
+<wire x1="81.28" y1="119.38" x2="71.12" y2="119.38" width="0.1524" layer="91"/>
+<pinref part="C100" gate="G$1" pin="8"/>
 </segment>
 <segment>
-<wire x1="81.28" y1="119.38" x2="71.12" y2="119.38" width="0.1524" layer="91"/>
-<pinref part="C100" gate="G$1" pin="8"/>
+<wire x1="154.94" y1="96.52" x2="144.78" y2="96.52" width="0.1524" layer="91"/>
+<pinref part="U1" gate="G$1" pin="P0_6"/>
 </segment>
 </net>
 <net name="RXD_MOSI" class="0">
 <segment>
-<pinref part="U1" gate="G$1" pin="P0_4"/>
-<wire x1="144.78" y1="101.6" x2="152.4" y2="101.6" width="0.1524" layer="91"/>
+<wire x1="81.28" y1="93.98" x2="71.12" y2="93.98" width="0.1524" layer="91"/>
+<pinref part="C100" gate="G$1" pin="3"/>
 </segment>
 <segment>
-<wire x1="81.28" y1="93.98" x2="71.12" y2="93.98" width="0.1524" layer="91"/>
-<pinref part="C100" gate="G$1" pin="3"/>
+<wire x1="154.94" y1="101.6" x2="144.78" y2="101.6" width="0.1524" layer="91"/>
+<pinref part="U1" gate="G$1" pin="P0_4"/>
 </segment>
 </net>
 <net name="!CS!" class="0">
 <segment>
-<wire x1="144.78" y1="93.98" x2="152.4" y2="93.98" width="0.1524" layer="91"/>
-<pinref part="U1" gate="G$1" pin="P0_7"/>
+<wire x1="81.28" y1="88.9" x2="71.12" y2="88.9" width="0.1524" layer="91"/>
+<pinref part="C100" gate="G$1" pin="2"/>
 </segment>
 <segment>
-<wire x1="81.28" y1="88.9" x2="71.12" y2="88.9" width="0.1524" layer="91"/>
-<pinref part="C100" gate="G$1" pin="2"/>
+<wire x1="154.94" y1="111.76" x2="144.78" y2="111.76" width="0.1524" layer="91"/>
+<pinref part="U1" gate="G$1" pin="P0_0"/>
 </segment>
 </net>
 <net name="DAT2" class="0">
 <segment>
-<pinref part="U1" gate="G$1" pin="P0_6"/>
-<wire x1="144.78" y1="96.52" x2="152.4" y2="96.52" width="0.1524" layer="91"/>
+<wire x1="81.28" y1="83.82" x2="71.12" y2="83.82" width="0.1524" layer="91"/>
+<pinref part="C100" gate="G$1" pin="1"/>
 </segment>
 <segment>
-<wire x1="81.28" y1="83.82" x2="71.12" y2="83.82" width="0.1524" layer="91"/>
-<pinref part="C100" gate="G$1" pin="1"/>
+<wire x1="154.94" y1="109.22" x2="144.78" y2="109.22" width="0.1524" layer="91"/>
+<pinref part="U1" gate="G$1" pin="P0_1"/>
 </segment>
 </net>
@@
 <pinref part="TP7" gate="G$1" pin="TP"/>
 <wire x1="144.78" y1="104.14" x2="182.88" y2="104.14" width="0.1524" layer="91"/>
-<label x="152.4" y="104.14" size="1.778" layer="95"/>
+<label x="154.94" y="104.14" size="1.778" layer="95"/>
 </segment>
 </net>
 <net name="SCK" class="0">
 <segment>
-<pinref part="U1" gate="G$1" pin="P0_5"/>
-<wire x1="144.78" y1="99.06" x2="152.4" y2="99.06" width="0.1524" layer="91"/>
+<wire x1="81.28" y1="104.14" x2="71.12" y2="104.14" width="0.1524" layer="91"/>
+<pinref part="C100" gate="G$1" pin="5"/>
 </segment>
 <segment>
-<wire x1="81.28" y1="104.14" x2="71.12" y2="104.14" width="0.1524" layer="91"/>
-<pinref part="C100" gate="G$1" pin="5"/>
+<wire x1="154.94" y1="99.06" x2="144.78" y2="99.06" width="0.1524" layer="91"/>
+<pinref part="U1" gate="G$1" pin="P0_5"/>
 </segment>
 </net>
@@
 <pinref part="U1" gate="G$1" pin="P0_2"/>
 <wire x1="182.88" y1="106.68" x2="144.78" y2="106.68" width="0.1524" layer="91"/>
-<label x="152.4" y="106.68" size="1.778" layer="95"/>
+<label x="154.94" y="106.68" size="1.778" layer="95"/>
 </segment>
 </net>
