File: MurataMicroSD.sch (EAGLE design)
At the start: 17 parts, among them CON1 CON_TC2030-CTL-NL, IC1 1265-1139-1-ND, U1 IC_BLE_LBCA2HNZYZ-711

Commit message: [ FIX ] library update
Parts:
- IC1: value 1265-1139-1-ND -> AT25XE011_TSSOP; device mylib:IC_SRAM_23K256_256K_32KBST -> mylib:IC_MEMORY_8P_AT25XE011_TSSOP
- TP100, TP101, TP102: value TPTP20R -> TESTPAD_F; device testpad_local:TPTP20R -> mylib:TESTPAD_F
Connections:
- net 3.3V renamed VCC
Other:
- moved on the sheet: C2
Changed lines of the file:
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@@
 <part name="R1" library="mylib" deviceset="R_US_PAD_PAD" device="_1005" value="10k/1005"/>
 <part name="SUPPLY3" library="mylib" deviceset="GND" device=""/>
-<part name="TP100" library="testpad_local" deviceset="TP" device="TP20R" value="TPTP20R"/>
-<part name="TP101" library="testpad_local" deviceset="TP" device="TP20R" value="TPTP20R"/>
-<part name="TP102" library="testpad_local" deviceset="TP" device="TP20R" value="TPTP20R"/>
+<part name="TP100" library="mylib" deviceset="TESTPAD" device="_F" value="TESTPAD_F"/>
+<part name="TP101" library="mylib" deviceset="TESTPAD" device="_F" value="TESTPAD_F"/>
+<part name="TP102" library="mylib" deviceset="TESTPAD" device="_F" value="TESTPAD_F"/>
 <part name="TP7" library="testpad_local" deviceset="TP" device="TP08R"/>
 <part name="TP8" library="testpad_local" deviceset="TP" device="TP08R"/>
@@
 <part name="SUPPLY4" library="mylib" deviceset="GND" device=""/>
 <part name="TP1" library="testpad_local" deviceset="TP" device="TP08R"/>
-<part name="IC1" library="mylib" deviceset="IC_SRAM_23K256_256K_32KB" device="ST" value="1265-1139-1-ND"/>
+<part name="IC1" library="mylib" deviceset="IC_MEMORY_8P_*" device="_TSSOP" technology="AT25XE011" value="AT25XE011_TSSOP"/>
 <part name="SUPPLY5" library="mylib" deviceset="GND" device=""/>
 <part name="C2" library="mylib" deviceset="C_PAD_PAD_" device="1005" value="0.1u/1005"/>
-<part name="SUPPLY6" library="mylib" deviceset="GND" device=""/>
 <part name="U$1" library="mylib" deviceset="ICON_OSHW" device=""/>
+<part name="P+1" library="mylib" deviceset="VCC" device=""/>
+<part name="P+3" library="mylib" deviceset="VCC" device=""/>
+<part name="P+4" library="mylib" deviceset="VCC" device=""/>
+<part name="P+5" library="mylib" deviceset="VCC" device=""/>
 </parts>
 <sheets>
@@
 <instance part="R1" gate="G$1" x="81.28" y="119.38"/>
 <instance part="SUPPLY3" gate="GND" x="73.66" y="119.38" rot="R270"/>
-<instance part="TP100" gate="G$1" x="231.14" y="43.18"/>
-<instance part="TP101" gate="G$1" x="238.76" y="43.18"/>
-<instance part="TP102" gate="G$1" x="246.38" y="43.18"/>
+<instance part="TP100" gate="1" x="231.14" y="43.18"/>
+<instance part="TP101" gate="1" x="238.76" y="43.18"/>
+<instance part="TP102" gate="1" x="246.38" y="43.18"/>
 <instance part="TP7" gate="G$1" x="160.02" y="109.22" rot="R270"/>
 <instance part="TP8" gate="G$1" x="162.56" y="111.76" rot="R270"/>
@@
 <instance part="SUPPLY4" gate="GND" x="154.94" y="121.92" rot="R270"/>
 <instance part="TP1" gate="G$1" x="149.86" y="101.6" rot="R270"/>
-<instance part="IC1" gate="G$1" x="195.58" y="99.06"/>
-<instance part="SUPPLY5" gate="GND" x="200.66" y="86.36"/>
-<instance part="C2" gate="G$1" x="208.28" y="114.3" rot="R90"/>
-<instance part="SUPPLY6" gate="GND" x="213.36" y="111.76"/>
+<instance part="IC1" gate="G$1" x="195.58" y="99.06" smashed="yes">
+<attribute name="NAME" x="182.88" y="110.39" size="1.778" layer="95"/>
+<attribute name="VALUE" x="182.88" y="88.8" size="1.778" layer="96"/>
+</instance>
+<instance part="SUPPLY5" gate="GND" x="210.82" y="99.06"/>
+<instance part="C2" gate="G$1" x="213.36" y="104.14"/>
 <instance part="U$1" gate="G$1" x="205.74" y="20.32"/>
+<instance part="P+1" gate="VCC" x="177.8" y="111.76"/>
+<instance part="P+3" gate="VCC" x="213.36" y="111.76"/>
+<instance part="P+4" gate="VCC" x="149.86" y="127" smashed="yes" rot="R90"/>
+<instance part="P+5" gate="VCC" x="68.58" y="114.3" smashed="yes" rot="R90"/>
 </instances>
 <busses>
 </busses>
 <nets>
-<net name="3.3V" class="0">
+<net name="VCC" class="0">
 <segment>
 <pinref part="C100" gate="G$1" pin="4"/>
@@
 <wire x1="86.36" y1="114.3" x2="88.9" y2="114.3" width="0.1524" layer="91"/>
 <junction x="86.36" y="114.3"/>
+<pinref part="P+5" gate="VCC" pin="VCC"/>
 </segment>
 <segment>
-<wire x1="157.48" y1="127" x2="147.32" y2="127" width="0.1524" layer="91"/>
+<wire x1="157.48" y1="127" x2="152.4" y2="127" width="0.1524" layer="91"/>
 <pinref part="CON1" gate="G$1" pin="VCC"/>
-<label x="147.32" y="127" size="1.778" layer="95"/>
+<label x="152.4" y="127" size="1.778" layer="95"/>
+<pinref part="P+4" gate="VCC" pin="VCC"/>
 </segment>
 <segment>
-<wire x1="200.66" y1="119.38" x2="200.66" y2="114.3" width="0.1524" layer="91"/>
 <pinref part="IC1" gate="G$1" pin="VCC"/>
-<wire x1="205.74" y1="114.3" x2="200.66" y2="114.3" width="0.1524" layer="91"/>
-<wire x1="200.66" y1="111.76" x2="200.66" y2="114.3" width="0.1524" layer="91"/>
-<wire x1="200.66" y1="114.3" x2="177.8" y2="114.3" width="0.1524" layer="91"/>
-<wire x1="177.8" y1="114.3" x2="177.8" y2="106.68" width="0.1524" layer="91"/>
+<pinref part="P+3" gate="VCC" pin="VCC"/>
+<wire x1="213.36" y1="109.22" x2="213.36" y2="106.68" width="0.1524" layer="91"/>
+<pinref part="C2" gate="G$1" pin="1"/>
+<junction x="213.36" y="106.68"/>
+<wire x1="213.36" y1="106.68" x2="208.28" y2="106.68" width="0.1524" layer="91"/>
+</segment>
+<segment>
+<wire x1="177.8" y1="109.22" x2="177.8" y2="106.68" width="0.1524" layer="91"/>
 <pinref part="IC1" gate="G$1" pin="!WP"/>
 <wire x1="177.8" y1="106.68" x2="180.34" y2="106.68" width="0.1524" layer="91"/>
@@
 <wire x1="177.8" y1="93.98" x2="177.8" y2="106.68" width="0.1524" layer="91"/>
 <junction x="177.8" y="106.68"/>
-<label x="200.66" y="119.38" size="1.778" layer="95"/>
-<pinref part="C2" gate="G$1" pin="1"/>
-<junction x="200.66" y="114.3"/>
+<pinref part="P+1" gate="VCC" pin="VCC"/>
 </segment>
 </net>
@@
 <pinref part="IC1" gate="G$1" pin="GND"/>
 <pinref part="SUPPLY5" gate="GND" pin="GND"/>
-</segment>
-<segment>
+<wire x1="210.82" y1="101.6" x2="208.28" y2="101.6" width="0.1524" layer="91"/>
 <pinref part="C2" gate="G$1" pin="2"/>
-<pinref part="SUPPLY6" gate="GND" pin="GND"/>
-<wire x1="210.82" y1="114.3" x2="213.36" y2="114.3" width="0.1524" layer="91"/>
+<wire x1="210.82" y1="101.6" x2="213.36" y2="101.6" width="0.1524" layer="91"/>
+<junction x="210.82" y="101.6"/>
 </segment>
 </net>
@@
 </segment>
 <segment>
-<wire x1="218.44" y1="99.06" x2="208.28" y2="99.06" width="0.1524" layer="91"/>
-<label x="218.44" y="99.06" size="1.778" layer="95"/>
+<wire x1="218.44" y1="93.98" x2="208.28" y2="93.98" width="0.1524" layer="91"/>
+<label x="218.44" y="93.98" size="1.778" layer="95"/>
 <pinref part="IC1" gate="G$1" pin="SO"/>
 </segment>

Commit message: [ uSD ] library update
Parts:
- C1, C2: device mylib:C_PAD_PAD_1005 -> mylib:C_SMD_0.1U_1005
- R1: device mylib:R_US_PAD_PAD_1005 -> mylib:R_US_10K_1005
Changed lines of the file:
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@@
 <part name="SUPPLY1" library="mylib" deviceset="GND" device=""/>
 <part name="SUPPLY2" library="mylib" deviceset="GND" device=""/>
-<part name="C1" library="mylib" deviceset="C_PAD_PAD_" device="1005" value="0.1u/1005"/>
-<part name="R1" library="mylib" deviceset="R_US_PAD_PAD" device="_1005" value="10k/1005"/>
+<part name="C1" library="mylib" deviceset="C_SMD_*" device="_1005" technology="0.1U" value="0.1u/1005"/>
+<part name="R1" library="mylib" deviceset="R_US_*" device="_1005" technology="10K" value="10k/1005"/>
 <part name="SUPPLY3" library="mylib" deviceset="GND" device=""/>
 <part name="TP100" library="mylib" deviceset="TESTPAD" device="_F" value="TESTPAD_F"/>
@@
 <part name="IC1" library="mylib" deviceset="IC_MEMORY_8P_*" device="_TSSOP" technology="AT25XE011" value="AT25XE011_TSSOP"/>
 <part name="SUPPLY5" library="mylib" deviceset="GND" device=""/>
-<part name="C2" library="mylib" deviceset="C_PAD_PAD_" device="1005" value="0.1u/1005"/>
+<part name="C2" library="mylib" deviceset="C_SMD_*" device="_1005" technology="0.1U" value="0.1u/1005"/>
 <part name="U$1" library="mylib" deviceset="ICON_OSHW" device=""/>
 <part name="P+1" library="mylib" deviceset="VCC" device=""/>
