File: MurataBLE_FS.sch (EAGLE design)
At the start: 51 parts, among them CON1 WM17143CT-ND, CON2 C-2395.microSD, IC1 74LVC1G00DBV, IC2 IC_DCDC_LM27313, IC3 IC_LPC11U3XQFN33, IC4 IC_LDO_XX1117_4, IC5 IC_MEMORY_8P_AT25XE011_TSSOP, SW1 SW_TACTSW_2PP8073, SW2 SW_TACTSW_2PP8073, SW3 SW_TACTSW_2PP8073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

Commit message: [ FS ] library update
Parts:
- C1, C10, C11, C16, C2: device mylib:C_PAD_PAD_1005 -> mylib:C_SMD_0.1U_1005
- C12, C13, C14, C3: device mylib:C_PAD_PAD_1005 -> mylib:C_SMD_18P_1005
- C15, C7: device mylib:C_PAD_PAD_1608 -> mylib:C_SMD_0.1U_1608
- C4, C5: device mylib:C_PAD_PAD_2125 -> mylib:C_SMD_4.7U_2012
- C6: device mylib:C_PAD_PAD_1608 -> mylib:C_SMD__1608
- C8, C9: value 4.7u/1608 -> 4.7u/2012; device mylib:C_PAD_PAD_2125 -> mylib:C_SMD_4.7U_2012
- L1: device mylib:INDUCTOR_2016 -> mylib:INDUCTOR_4.7U_2016
- R1, R10: device mylib:R_US_PAD_PAD_1005 -> mylib:R_US_33R_1005
- R11: device mylib:R_US_PAD_PAD_1005 -> mylib:R_US_1.5K_1005
- R12, R7, R8, R9: device mylib:R_US_PAD_PAD_1005 -> mylib:R_US_10K_1005
- R13, R14: device mylib:R_US_PAD_PAD_1005 -> mylib:R_US_100R_1005
- R2: device mylib:R_US_PAD_PAD_1608 -> mylib:R_US_10K_1608
- R3: device mylib:R_US_PAD_PAD_1608 -> mylib:R_US_60.4K_1608
- R4: device mylib:R_US_PAD_PAD_1608 -> mylib:R_US_13.3K_1608
- R5, R6: value 100/1005 -> 1k/1005; device mylib:R_US_PAD_PAD_1005 -> mylib:R_US_1.0K_1005
Changed lines of the file:
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@@
 <part name="SUPPLY1" library="mylib" deviceset="GND" device=""/>
 <part name="SUPPLY3" library="mylib" deviceset="GND" device=""/>
-<part name="C1" library="mylib" deviceset="C_PAD_PAD_" device="1005" value="0.1u"/>
+<part name="C1" library="mylib" deviceset="C_SMD_*" device="_1005" technology="0.1U" value="0.1u"/>
 <part name="SUPPLY6" library="mylib" deviceset="GND" device=""/>
-<part name="C2" library="mylib" deviceset="C_PAD_PAD_" device="1005" value="0.1u"/>
-<part name="L1" library="mylib" deviceset="INDUCTOR" device="_2016" value="4.7uH/2016"/>
+<part name="C2" library="mylib" deviceset="C_SMD_*" device="_1005" technology="0.1U" value="0.1u"/>
+<part name="L1" library="mylib" deviceset="INDUCTOR_" device="_2016" technology="4.7U" value="4.7uH/2016"/>
 <part name="IC2" library="mylib" deviceset="IC_DCDC_LM27313" device=""/>
 <part name="D1" library="mylib" deviceset="DIODE_SMALL" device=""/>
-<part name="R2" library="mylib" deviceset="R_US_PAD_PAD" device="_1608" value="10k"/>
-<part name="R3" library="mylib" deviceset="R_US_PAD_PAD" device="_1608" value="60.4k"/>
-<part name="R4" library="mylib" deviceset="R_US_PAD_PAD" device="_1608" value="13.3k"/>
-<part name="C4" library="mylib" deviceset="C_PAD_PAD_" device="2125" value="4.7u"/>
-<part name="C5" library="mylib" deviceset="C_PAD_PAD_" device="2125" value="4.7u"/>
-<part name="C6" library="mylib" deviceset="C_PAD_PAD_" device="1608" value="NM"/>
+<part name="R2" library="mylib" deviceset="R_US_*" device="_1608" technology="10K" value="10k"/>
+<part name="R3" library="mylib" deviceset="R_US_*" device="_1608" technology="60.4K" value="60.4k"/>
+<part name="R4" library="mylib" deviceset="R_US_*" device="_1608" technology="13.3K" value="13.3k"/>
+<part name="C4" library="mylib" deviceset="C_SMD_*" device="_2012" technology="4.7U" value="4.7u"/>
+<part name="C5" library="mylib" deviceset="C_SMD_*" device="_2012" technology="4.7U" value="4.7u"/>
+<part name="C6" library="mylib" deviceset="C_SMD_*" device="_1608" value="NM"/>
 <part name="SUPPLY10" library="mylib" deviceset="GND" device=""/>
 <part name="SUPPLY11" library="mylib" deviceset="GND" device=""/>
 <part name="X1" library="con-samtec.local" deviceset="TSW-102-02-S-S" device=""/>
-<part name="C7" library="mylib" deviceset="C_PAD_PAD_" device="1608" value="0.1u"/>
+<part name="C7" library="mylib" deviceset="C_SMD_*" device="_1608" technology="0.1U" value="0.1u"/>
 <part name="TP1" library="testpad_local" deviceset="TP" device="PAD1-13" value="P7592"/>
 <part name="TP2" library="testpad_local" deviceset="TP" device="PAD1-13" value="P7591"/>
 <part name="IC3" library="mylib" deviceset="IC_LPC11U3XQFN33" device=""/>
-<part name="C8" library="mylib" deviceset="C_PAD_PAD_" device="2125" value="4.7u/1608"/>
-<part name="C9" library="mylib" deviceset="C_PAD_PAD_" device="2125" value="4.7u/1608"/>
+<part name="C8" library="mylib" deviceset="C_SMD_*" device="_2012" technology="4.7U" value="4.7u/2012"/>
+<part name="C9" library="mylib" deviceset="C_SMD_*" device="_2012" technology="4.7U" value="4.7u/2012"/>
 <part name="SUPPLY12" library="mylib" deviceset="GND" device=""/>
 <part name="SUPPLY13" library="mylib" deviceset="GND" device=""/>
-<part name="C10" library="mylib" deviceset="C_PAD_PAD_" device="1005" value="0.1u"/>
-<part name="C11" library="mylib" deviceset="C_PAD_PAD_" device="1005" value="0.1u"/>
-<part name="R5" library="mylib" deviceset="R_US_PAD_PAD" device="_1005" value="100/1005"/>
-<part name="R6" library="mylib" deviceset="R_US_PAD_PAD" device="_1005" value="100/1005"/>
-<part name="R7" library="mylib" deviceset="R_US_PAD_PAD" device="_1005" value="10k/1005"/>
-<part name="R8" library="mylib" deviceset="R_US_PAD_PAD" device="_1005" value="10k/1005"/>
-<part name="R9" library="mylib" deviceset="R_US_PAD_PAD" device="_1005" value="10k/1005"/>
+<part name="C10" library="mylib" deviceset="C_SMD_*" device="_1005" technology="0.1U" value="0.1u"/>
+<part name="C11" library="mylib" deviceset="C_SMD_*" device="_1005" technology="0.1U" value="0.1u"/>
+<part name="R5" library="mylib" deviceset="R_US_*" device="_1005" technology="1.0K" value="1k/1005"/>
+<part name="R6" library="mylib" deviceset="R_US_*" device="_1005" technology="1.0K" value="1k/1005"/>
+<part name="R7" library="mylib" deviceset="R_US_*" device="_1005" technology="10K" value="10k/1005"/>
+<part name="R8" library="mylib" deviceset="R_US_*" device="_1005" technology="10K" value="10k/1005"/>
+<part name="R9" library="mylib" deviceset="R_US_*" device="_1005" technology="10K" value="10k/1005"/>
 <part name="Q1" library="mylib" deviceset="CLOCK_CRYSTAL_4" device="_3225"/>
-<part name="C3" library="mylib" deviceset="C_PAD_PAD_" device="1005" value="18p/1005"/>
-<part name="C12" library="mylib" deviceset="C_PAD_PAD_" device="1005" value="18p/1005"/>
+<part name="C3" library="mylib" deviceset="C_SMD_*" device="_1005" technology="18P" value="18p/1005"/>
+<part name="C12" library="mylib" deviceset="C_SMD_*" device="_1005" technology="18P" value="18p/1005"/>
 <part name="SUPPLY2" library="mylib" deviceset="GND" device=""/>
 <part name="IC4" library="mylib" deviceset="IC_LDO_XX1117_4" device=""/>
-<part name="R1" library="mylib" deviceset="R_US_PAD_PAD" device="_1005" value="33/1005"/>
-<part name="R10" library="mylib" deviceset="R_US_PAD_PAD" device="_1005" value="33/1005"/>
-<part name="C13" library="mylib" deviceset="C_PAD_PAD_" device="1005" value="18p/1005"/>
-<part name="C14" library="mylib" deviceset="C_PAD_PAD_" device="1005" value="18p/1005"/>
+<part name="R1" library="mylib" deviceset="R_US_*" device="_1005" technology="33R" value="33/1005"/>
+<part name="R10" library="mylib" deviceset="R_US_*" device="_1005" technology="33R" value="33/1005"/>
+<part name="C13" library="mylib" deviceset="C_SMD_*" device="_1005" technology="18P" value="18p/1005"/>
+<part name="C14" library="mylib" deviceset="C_SMD_*" device="_1005" technology="18P" value="18p/1005"/>
 <part name="TR1" library="mylib" deviceset="TR_PMOS_GDS" device="_SOT23" value="I-4269"/>
-<part name="R11" library="mylib" deviceset="R_US_PAD_PAD" device="_1005" value="1.5k/1005"/>
+<part name="R11" library="mylib" deviceset="R_US_*" device="_1005" technology="1.5K" value="1.5k/1005"/>
 <part name="SUPPLY9" library="mylib" deviceset="GND" device=""/>
 <part name="SUPPLY14" library="mylib" deviceset="GND" device=""/>
-<part name="R12" library="mylib" deviceset="R_US_PAD_PAD" device="_1005" value="10k/1005"/>
+<part name="R12" library="mylib" deviceset="R_US_*" device="_1005" technology="10K" value="10k/1005"/>
 <part name="SUPPLY15" library="mylib" deviceset="GND" device=""/>
 <part name="SW1" library="mylib" deviceset="SW_TACTSW_2P" device="P8073"/>
@@
 <part name="CON2" library="mylib" deviceset="CON_MICROSD" device="_C2395" value="C-2395.microSD"/>
 <part name="SUPPLY19" library="mylib" deviceset="GND" device=""/>
-<part name="C15" library="mylib" deviceset="C_PAD_PAD_" device="1608" value="0.1u"/>
+<part name="C15" library="mylib" deviceset="C_SMD_*" device="_1608" technology="0.1U" value="0.1u"/>
 <part name="SUPPLY20" library="mylib" deviceset="GND" device=""/>
 <part name="SUPPLY21" library="mylib" deviceset="GND" device=""/>
@@
 <part name="IC5" library="mylib" deviceset="IC_MEMORY_8P_*" device="_TSSOP" technology="AT25XE011" value="IC_MEMORY_8P_AT25XE011_TSSOP"/>
 <part name="SUPPLY25" library="mylib" deviceset="GND" device=""/>
-<part name="C16" library="mylib" deviceset="C_PAD_PAD_" device="1005" value="0.1u"/>
-<part name="R13" library="mylib" deviceset="R_US_PAD_PAD" device="_1005" value="100/1005"/>
-<part name="R14" library="mylib" deviceset="R_US_PAD_PAD" device="_1005" value="100/1005"/>
+<part name="C16" library="mylib" deviceset="C_SMD_*" device="_1005" technology="0.1U" value="0.1u"/>
+<part name="R13" library="mylib" deviceset="R_US_*" device="_1005" technology="100R" value="100/1005"/>
+<part name="R14" library="mylib" deviceset="R_US_*" device="_1005" technology="100R" value="100/1005"/>
 <part name="LED1" library="mylib" deviceset="LED_1SEG_A2K1" device=""/>
 <part name="SUPPLY5" library="mylib" deviceset="GND" device=""/>
