File: MurataBLE_FS.sch (EAGLE design)
At the start: 51 parts, among them CON1 WM17143CT-ND, CON2 C-2395.microSD, IC1 74LVC1G00DBV, IC2 IC_DCDC_LM27313, IC3 IC_LPC11U3XQFN33, IC4 IC_LDO_XX1117_4, IC5 IC_MEMORY_8P_AT25XE011_TSSOP, SW1 SW_TACTSW_2PP8073, SW2 SW_TACTSW_2PP8073, SW3 SW_TACTSW_2PP8073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

Commit message: update eagle version = 7.5.0; library update
Parts:
- CON1: device mylib:CON_USBMICROBUB -> mylib:CON_USB_UB
- IC4: value IC_LDO_XX1117_4 -> LDO4_3.3_SOT223; device mylib:IC_LDO_XX1117_4 -> mylib:LDO4_3.3_SOT223
- Q1: device mylib:CLOCK_CRYSTAL_4_3225 -> mylib:CRYSTAL4_12M_3225
- SW1, SW3: value SW_TACTSW_2PP8073 -> (none); device mylib:SW_TACTSW_2PP8073 -> mylib:TACTSW2_BK_P807X
- SW2: value SW_TACTSW_2PP8073 -> (none); device mylib:SW_TACTSW_2PP8073 -> mylib:TACTSW2_WH_P807X
- U1: value IC_BLE_LBCA2HNZYZ-711 -> LBCA2HNZYZ-711; device mylib:IC_BLE_LBCA2HNZYZ-711 -> mylib:LBCA2HNZYZ-711
Connections:
- net VCC: now also IC4.OUT/EN/NC; no longer IC4.OUT@1
Other:
- moved on the sheet: CON1, IC2, IC4
Changed lines of the file:
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@@
 <?xml version="1.0" encoding="utf-8"?>
 <!DOCTYPE eagle SYSTEM "eagle.dtd">
-<eagle version="6.5.0">
+<eagle version="7.5.0">
 <drawing>
 <settings>
@@
 <part name="PCB1" library="dp_pcb_local" deviceset="PCB_DP_RECTANGLE" device="-43X70" value="PCB_DP_RECTANGLE-43X70"/>
 <part name="IC1" library="74xx-little-us_local" deviceset="74*1G00" device="DBV" technology="LVC"/>
-<part name="CON1" library="mylib" deviceset="CON_USB" device="UB" technology="MICROB" value="WM17143CT-ND"/>
+<part name="CON1" library="mylib" deviceset="CON_USB" device="_UB" value="WM17143CT-ND"/>
 <part name="SUPPLY1" library="mylib" deviceset="GND" device=""/>
 <part name="SUPPLY3" library="mylib" deviceset="GND" device=""/>
@@
 <part name="R8" library="mylib" deviceset="R_US_*" device="_1005" technology="10K" value="10k/1005"/>
 <part name="R9" library="mylib" deviceset="R_US_*" device="_1005" technology="10K" value="10k/1005"/>
-<part name="Q1" library="mylib" deviceset="CLOCK_CRYSTAL_4" device="_3225"/>
+<part name="Q1" library="mylib" deviceset="CRYSTAL4_*" device="_3225" technology="12M"/>
 <part name="C3" library="mylib" deviceset="C_SMD_*" device="_1005" technology="18P" value="18p/1005"/>
 <part name="C12" library="mylib" deviceset="C_SMD_*" device="_1005" technology="18P" value="18p/1005"/>
 <part name="SUPPLY2" library="mylib" deviceset="GND" device=""/>
-<part name="IC4" library="mylib" deviceset="IC_LDO_XX1117_4" device=""/>
 <part name="R1" library="mylib" deviceset="R_US_*" device="_1005" technology="33R" value="33/1005"/>
 <part name="R10" library="mylib" deviceset="R_US_*" device="_1005" technology="33R" value="33/1005"/>
@@
 <part name="R12" library="mylib" deviceset="R_US_*" device="_1005" technology="10K" value="10k/1005"/>
 <part name="SUPPLY15" library="mylib" deviceset="GND" device=""/>
-<part name="SW1" library="mylib" deviceset="SW_TACTSW_2P" device="P8073"/>
-<part name="SW2" library="mylib" deviceset="SW_TACTSW_2P" device="P8073"/>
-<part name="SW3" library="mylib" deviceset="SW_TACTSW_2P" device="P8073"/>
+<part name="SW1" library="mylib" deviceset="TACTSW2_*" device="_P807X" technology="BK"/>
+<part name="SW2" library="mylib" deviceset="TACTSW2_*" device="_P807X" technology="WH"/>
+<part name="SW3" library="mylib" deviceset="TACTSW2_*" device="_P807X" technology="BK"/>
 <part name="SUPPLY16" library="mylib" deviceset="GND" device=""/>
 <part name="SUPPLY17" library="mylib" deviceset="GND" device=""/>
@@
 <part name="U$1" library="mylib" deviceset="ICON_OSHW" device=""/>
 <part name="SUPPLY22" library="mylib" deviceset="GND" device=""/>
-<part name="U1" library="mylib" deviceset="IC_BLE_LBCA2HNZYZ-711" device=""/>
+<part name="U1" library="mylib" deviceset="LBCA2HNZYZ-711" device=""/>
 <part name="FRAME2" library="frames" deviceset="A4L-LOC" device=""/>
 <part name="SUPPLY24" library="mylib" deviceset="GND" device=""/>
@@
 <part name="P+7" library="mylib" deviceset="VCC" device=""/>
 <part name="P+8" library="mylib" deviceset="VCC" device=""/>
+<part name="IC4" library="mylib" deviceset="LDO4_*" device="_SOT223" technology="3.3"/>
 </parts>
 <sheets>
@@
 <instance part="C2" gate="G$1" x="66.04" y="-83.82"/>
 <instance part="L1" gate="G$1" x="73.66" y="40.64"/>
-<instance part="IC2" gate="G$1" x="73.66" y="27.94"/>
+<instance part="IC2" gate="G$1" x="73.66" y="22.86"/>
 <instance part="D1" gate="G$1" x="91.44" y="40.64"/>
 <instance part="R2" gate="G$1" x="55.88" y="35.56" rot="R90"/>
@@
 <instance part="C12" gate="G$1" x="104.14" y="99.06" rot="MR0"/>
 <instance part="SUPPLY2" gate="GND" x="104.14" y="86.36"/>
-<instance part="IC4" gate="G$1" x="45.72" y="71.12" smashed="yes">
-<attribute name="NAME" x="48.26" y="63.5" size="1.778" layer="95"/>
-<attribute name="VALUE" x="40.64" y="74.93" size="1.016" layer="96"/>
-</instance>
 <instance part="R1" gate="G$1" x="55.88" y="134.62"/>
 <instance part="R10" gate="G$1" x="55.88" y="137.16"/>
@@
 <instance part="P+7" gate="VCC" x="48.26" y="172.72"/>
 <instance part="P+8" gate="VCC" x="63.5" y="-78.74"/>
+<instance part="IC4" gate="G$1" x="45.72" y="71.12"/>
 </instances>
 <busses>
@@
 </segment>
 <segment>
-<pinref part="IC2" gate="G$1" pin="GND"/>
 <pinref part="C4" gate="G$1" pin="2"/>
-<wire x1="60.96" y1="22.86" x2="50.8" y2="22.86" width="0.1524" layer="91"/>
+<pinref part="C7" gate="G$1" pin="2"/>
+<wire x1="50.8" y1="27.94" x2="50.8" y2="22.86" width="0.1524" layer="91"/>
 <wire x1="50.8" y1="22.86" x2="45.72" y2="22.86" width="0.1524" layer="91"/>
 <wire x1="45.72" y1="22.86" x2="45.72" y2="27.94" width="0.1524" layer="91"/>
+<junction x="45.72" y="22.86"/>
 <wire x1="45.72" y1="22.86" x2="45.72" y2="20.32" width="0.1524" layer="91"/>
-<junction x="45.72" y="22.86"/>
 <pinref part="SUPPLY10" gate="GND" pin="GND"/>
-<pinref part="C7" gate="G$1" pin="2"/>
-<wire x1="50.8" y1="27.94" x2="50.8" y2="22.86" width="0.1524" layer="91"/>
-<junction x="50.8" y="22.86"/>
 </segment>
 <segment>
@@
 <wire x1="109.22" y1="15.24" x2="121.92" y2="15.24" width="0.1524" layer="91"/>
 <junction x="109.22" y="15.24"/>
+<wire x1="101.6" y1="15.24" x2="91.44" y2="15.24" width="0.1524" layer="91"/>
+<wire x1="91.44" y1="15.24" x2="91.44" y2="17.78" width="0.1524" layer="91"/>
+<pinref part="IC2" gate="G$1" pin="GND"/>
+<wire x1="91.44" y1="17.78" x2="86.36" y2="17.78" width="0.1524" layer="91"/>
 </segment>
 <segment>
@@
 <wire x1="58.42" y1="71.12" x2="58.42" y2="66.04" width="0.1524" layer="91"/>
 <junction x="58.42" y="71.12"/>
-<pinref part="IC4" gate="G$1" pin="OUT"/>
-<pinref part="IC4" gate="G$1" pin="OUT@1"/>
 <wire x1="53.34" y1="68.58" x2="55.88" y2="68.58" width="0.1524" layer="91"/>
 <wire x1="55.88" y1="68.58" x2="55.88" y2="71.12" width="0.1524" layer="91"/>
 <junction x="55.88" y="71.12"/>
 <pinref part="P+1" gate="VCC" pin="VCC"/>
+<pinref part="IC4" gate="G$1" pin="OUT"/>
+<pinref part="IC4" gate="G$1" pin="OUT/EN/NC"/>
+<wire x1="45.72" y1="76.2" x2="55.88" y2="76.2" width="0.1524" layer="91"/>
+<wire x1="55.88" y1="76.2" x2="55.88" y2="71.12" width="0.1524" layer="91"/>
 </segment>
 <segment>
@@
 <segment>
 <pinref part="CON1" gate="G$1" pin="SHLD"/>
-<junction x="12.7" y="129.54"/>
+<junction x="27.94" y="129.54"/>
 </segment>
 </net>
@@
 <wire x1="71.12" y1="40.64" x2="60.96" y2="40.64" width="0.1524" layer="91"/>
 <pinref part="IC2" gate="G$1" pin="VIN"/>
-<wire x1="60.96" y1="40.64" x2="60.96" y2="33.02" width="0.1524" layer="91"/>
+<wire x1="60.96" y1="40.64" x2="60.96" y2="27.94" width="0.1524" layer="91"/>
 <wire x1="60.96" y1="40.64" x2="55.88" y2="40.64" width="0.1524" layer="91"/>
 <junction x="60.96" y="40.64"/>
@@
 <pinref part="IC2" gate="G$1" pin="LX"/>
 <wire x1="76.2" y1="40.64" x2="86.36" y2="40.64" width="0.1524" layer="91"/>
-<wire x1="86.36" y1="40.64" x2="86.36" y2="33.02" width="0.1524" layer="91"/>
+<wire x1="86.36" y1="40.64" x2="86.36" y2="27.94" width="0.1524" layer="91"/>
 <pinref part="D1" gate="G$1" pin="A"/>
 <wire x1="86.36" y1="40.64" x2="88.9" y2="40.64" width="0.1524" layer="91"/>
@@
 <segment>
 <pinref part="IC2" gate="G$1" pin="!SHDN!"/>
-<wire x1="60.96" y1="27.94" x2="55.88" y2="27.94" width="0.1524" layer="91"/>
+<wire x1="60.96" y1="17.78" x2="55.88" y2="17.78" width="0.1524" layer="91"/>
 <pinref part="R2" gate="G$1" pin="1"/>
-<wire x1="55.88" y1="27.94" x2="55.88" y2="33.02" width="0.1524" layer="91"/>
-</segment>
-</net>
+<wire x1="55.88" y1="17.78" x2="55.88" y2="33.02" width="0.1524" layer="91"/>
+</segment>
+</net>
