File: DA14580_QFN40_0v5.sch (EAGLE design)
At the start: 26 parts, among them CON1 CON_TC2030-CTL-NL, IC1 IC_SRAM_23K256_256K_32KBSN, IC2 74LVC1G00DBV, IC3 IC_LDO_XX1117, U1 IC_DA14580_QFN40, X1 SSW-114-02-S-S, X2 SSW-114-02-S-S

Commit message: [ FIX ][ 58X ] update schematic with library
Parts:
- IC1: value IC_SRAM_23K256_256K_32KBSN -> IC_MEMORY_8P_AT25XE011_SOP; device mylib:IC_SRAM_23K256_256K_32KBSN -> mylib:IC_MEMORY_8P_AT25XE011_SOP
- IC3: value IC_LDO_XX1117 -> IC_LDO_XX1117_5; device mylib:IC_LDO_XX1117 -> mylib:IC_LDO_XX1117_5
- L1: value INDUCTOR_1608 -> 2.2u
- U1: value IC_DA14580_QFN40 -> DA14583-AT2; device mylib:IC_DA14580_QFN40 -> mylib:DA14583-AT2
Connections:
- net GND: no longer U1.BP
- net VCC: now also U1.NC/VDD_FLASH; no longer U1.NC
Other:
- note added: "L1: 445-6385-1-ND"
- moved on the sheet: C3, C4, L1, TP1
Changed lines of the file:
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@@
 <parts>
 <part name="FRAME1" library="frames" deviceset="A4L-LOC" device="" value="A4L-LOC"/>
-<part name="U1" library="mylib" deviceset="IC_DA14580_QFN40" device=""/>
+<part name="U1" library="mylib" deviceset="DA1458*" device="-AT2" technology="3" value="DA14583-AT2"/>
 <part name="SUPPLY1" library="mylib" deviceset="GND" device=""/>
 <part name="SUPPLY2" library="mylib" deviceset="GND" device=""/>
@@
 <part name="SUPPLY11" library="mylib" deviceset="GND" device=""/>
 <part name="C3" library="mylib" deviceset="C_PAD_PAD_" device="1005"/>
-<part name="L1" library="mylib" deviceset="INDUCTOR" device="_1608"/>
+<part name="L1" library="mylib" deviceset="INDUCTOR" device="_1608" value="2.2u"/>
 <part name="R1" library="mylib" deviceset="R_US_PAD_PAD" device="_1005"/>
-<part name="IC1" library="mylib" deviceset="IC_SRAM_23K256_256K_32KB" device="SN" value="IC_SRAM_23K256_256K_32KBSN"/>
-<part name="SUPPLY3" library="mylib" deviceset="GND" device=""/>
+<part name="IC1" library="mylib" deviceset="IC_MEMORY_8P_*" device="_SOP" technology="AT25XE011" value="IC_MEMORY_8P_AT25XE011_SOP"/>
 <part name="P+3" library="mylib" deviceset="VCC" device=""/>
 <part name="C4" library="mylib" deviceset="C_PAD_PAD_" device="1005"/>
@@
 <part name="TP3" library="testpad_local" deviceset="TP" device="TP07R" value="TPTP07R"/>
 <part name="P+5" library="mylib" deviceset="VCC" device=""/>
-<part name="IC3" library="mylib" deviceset="IC_LDO_XX1117" device=""/>
+<part name="IC3" library="mylib" deviceset="IC_LDO_XX1117_5" device=""/>
 <part name="IC2" library="74xx-little-us_local" deviceset="74*1G00" device="DBV" technology="LVC"/>
 <part name="TP6" library="testpad_local" deviceset="TP" device="PAD1-13"/>
@@
 <part name="C8" library="mylib" deviceset="C_PAD_PAD_" device="1005"/>
 <part name="C9" library="mylib" deviceset="C_PAD_PAD_" device="1005"/>
-<part name="SUPPLY14" library="mylib" deviceset="GND" device=""/>
 <part name="C10" library="mylib" deviceset="C_PAD_PAD_" device="1005"/>
 <part name="SUPPLY15" library="mylib" deviceset="GND" device=""/>
@@
 <part name="P+6" library="mylib" deviceset="VCC" device=""/>
 <part name="Q2" library="mylib" deviceset="CLOCK_CRYSTAL_4" device="_2520"/>
+<part name="P+7" library="mylib" deviceset="VCC" device=""/>
 </parts>
 <sheets>
@@
 <plain>
 <text x="217.17" y="25.4" size="12.7" layer="94">v0.5</text>
+<text x="12.7" y="167.64" size="1.778" layer="94">L1: 445-6385-1-ND</text>
 </plain>
 <instances>
 <instance part="FRAME1" gate="G$1" x="0" y="0"/>
 <instance part="U1" gate="G$1" x="104.14" y="142.24"/>
-<instance part="SUPPLY1" gate="GND" x="81.28" y="152.4"/>
+<instance part="SUPPLY1" gate="GND" x="81.28" y="154.94" rot="R270"/>
 <instance part="SUPPLY2" gate="GND" x="147.32" y="152.4"/>
 <instance part="SUPPLY4" gate="GND" x="210.82" y="33.02"/>
-<instance part="SUPPLY6" gate="GND" x="71.12" y="139.7"/>
+<instance part="SUPPLY6" gate="GND" x="68.58" y="142.24" rot="R270"/>
 <instance part="VDD1" gate="G$1" x="213.36" y="161.29"/>
 <instance part="P+1" gate="VCC" x="238.76" y="162.56"/>
@@
 <instance part="C2" gate="G$1" x="238.76" y="151.13"/>
 <instance part="SUPPLY9" gate="GND" x="238.76" y="142.24"/>
-<instance part="SUPPLY11" gate="GND" x="58.42" y="139.7"/>
-<instance part="C3" gate="G$1" x="58.42" y="147.32"/>
-<instance part="L1" gate="G$1" x="81.28" y="139.7"/>
+<instance part="SUPPLY11" gate="GND" x="53.34" y="139.7"/>
+<instance part="C3" gate="G$1" x="53.34" y="147.32"/>
+<instance part="L1" gate="G$1" x="76.2" y="139.7"/>
 <instance part="R1" gate="G$1" x="213.36" y="67.31" rot="R90"/>
 <instance part="IC1" gate="G$1" x="223.52" y="101.6"/>
-<instance part="SUPPLY3" gate="GND" x="228.6" y="86.36"/>
-<instance part="P+3" gate="VCC" x="228.6" y="119.38"/>
-<instance part="C4" gate="G$1" x="241.3" y="111.76"/>
-<instance part="SUPPLY13" gate="GND" x="241.3" y="104.14"/>
-<instance part="TP1" gate="G$1" x="76.2" y="152.4"/>
+<instance part="P+3" gate="VCC" x="205.74" y="114.3"/>
+<instance part="C4" gate="G$1" x="241.3" y="106.68"/>
+<instance part="SUPPLY13" gate="GND" x="241.3" y="101.6"/>
+<instance part="TP1" gate="G$1" x="63.5" y="152.4"/>
 <instance part="X1" gate="-1" x="86.36" y="60.96" rot="MR0"/>
 <instance part="X1" gate="-2" x="86.36" y="58.42" rot="MR0"/>
@@
 <instance part="C8" gate="G$1" x="124.46" y="157.48"/>
 <instance part="C9" gate="G$1" x="73.66" y="144.78"/>
-<instance part="SUPPLY14" gate="GND" x="71.12" y="93.98"/>
 <instance part="C10" gate="G$1" x="83.82" y="91.44"/>
 <instance part="SUPPLY15" gate="GND" x="83.82" y="86.36"/>
@@
 <attribute name="VALUE" x="66.802" y="129.54" size="1.016" layer="96" rot="R270"/>
 </instance>
+<instance part="P+7" gate="VCC" x="241.3" y="114.3"/>
 </instances>
 <busses>
@@
 <pinref part="U1" gate="G$1" pin="GND"/>
 <pinref part="SUPPLY1" gate="GND" pin="GND"/>
-<wire x1="86.36" y1="154.94" x2="81.28" y2="154.94" width="0.1524" layer="91"/>
+<wire x1="86.36" y1="154.94" x2="83.82" y2="154.94" width="0.1524" layer="91"/>
 </segment>
 <segment>
@@
 </segment>
 <segment>
-<pinref part="U1" gate="G$1" pin="BP"/>
-<wire x1="86.36" y1="96.52" x2="71.12" y2="96.52" width="0.1524" layer="91"/>
-<pinref part="SUPPLY14" gate="GND" pin="GND"/>
-</segment>
-<segment>
 <pinref part="U1" gate="G$1" pin="VBAT1V"/>
 <pinref part="SUPPLY6" gate="GND" pin="GND"/>
@@
 <pinref part="SUPPLY11" gate="GND" pin="GND"/>
 <pinref part="C3" gate="G$1" pin="2"/>
-<wire x1="58.42" y1="142.24" x2="58.42" y2="144.78" width="0.1524" layer="91"/>
+<wire x1="53.34" y1="142.24" x2="53.34" y2="144.78" width="0.1524" layer="91"/>
 </segment>
 <segment>
 <pinref part="IC1" gate="G$1" pin="GND"/>
-<pinref part="SUPPLY3" gate="GND" pin="GND"/>
-<wire x1="228.6" y1="91.44" x2="228.6" y2="88.9" width="0.1524" layer="91"/>
-</segment>
-<segment>
 <pinref part="C4" gate="G$1" pin="2"/>
 <pinref part="SUPPLY13" gate="GND" pin="GND"/>
-<wire x1="241.3" y1="106.68" x2="241.3" y2="109.22" width="0.1524" layer="91"/>
+<wire x1="236.22" y1="104.14" x2="241.3" y2="104.14" width="0.1524" layer="91"/>
+<junction x="241.3" y="104.14"/>
 </segment>
 <segment>
@@
 </segment>
 <segment>
+<pinref part="C4" gate="G$1" pin="1"/>
+<pinref part="P+7" gate="VCC" pin="VCC"/>
+<pinref part="IC1" gate="G$1" pin="VCC"/>
+<wire x1="236.22" y1="109.22" x2="241.3" y2="109.22" width="0.1524" layer="91"/>
+<wire x1="241.3" y1="111.76" x2="241.3" y2="109.22" width="0.1524" layer="91"/>
+<junction x="241.3" y="109.22"/>
+</segment>
+<segment>
 <pinref part="P+3" gate="VCC" pin="VCC"/>
-<pinref part="IC1" gate="G$1" pin="VCC"/>
-<wire x1="228.6" y1="114.3" x2="228.6" y2="116.84" width="0.1524" layer="91"/>
 <pinref part="IC1" gate="G$1" pin="!HOLD"/>
 <pinref part="IC1" gate="G$1" pin="!WP"/>
@@
 <wire x1="205.74" y1="96.52" x2="205.74" y2="109.22" width="0.1524" layer="91"/>
 <wire x1="205.74" y1="109.22" x2="208.28" y2="109.22" width="0.1524" layer="91"/>
-<wire x1="228.6" y1="116.84" x2="205.74" y2="116.84" width="0.1524" layer="91"/>
-<wire x1="205.74" y1="116.84" x2="205.74" y2="109.22" width="0.1524" layer="91"/>
-<junction x="228.6" y="116.84"/>
+<wire x1="205.74" y1="111.76" x2="205.74" y2="109.22" width="0.1524" layer="91"/>
 <junction x="205.74" y="109.22"/>
-<pinref part="C4" gate="G$1" pin="1"/>
-<wire x1="228.6" y1="116.84" x2="241.3" y2="116.84" width="0.1524" layer="91"/>
-<wire x1="241.3" y1="116.84" x2="241.3" y2="114.3" width="0.1524" layer="91"/>
 </segment>
 <segment>
@@
 </segment>
 <segment>
-<pinref part="U1" gate="G$1" pin="NC"/>
+<pinref part="U1" gate="G$1" pin="NC/VDD_FLASH"/>
 <pinref part="P+5" gate="VCC" pin="VCC"/>
 <wire x1="81.28" y1="93.98" x2="83.82" y2="93.98" width="0.1524" layer="91"/>
@@
 <pinref part="U1" gate="G$1" pin="LX"/>
 <pinref part="L1" gate="G$1" pin="2"/>
-<wire x1="86.36" y1="139.7" x2="83.82" y2="139.7" width="0.1524" layer="91"/>
+<wire x1="86.36" y1="139.7" x2="78.74" y2="139.7" width="0.1524" layer="91"/>
 </segment>
 </net>
@@
 </segment>
 <segment>
-<wire x1="236.22" y1="101.6" x2="250.19" y2="101.6" width="0.1524" layer="91"/>
-<label x="245.11" y="101.6" size="1.778" layer="95"/>
+<wire x1="236.22" y1="96.52" x2="245.11" y2="96.52" width="0.1524" layer="91"/>
+<label x="245.11" y="96.52" size="1.778" layer="95"/>
 <pinref part="IC1" gate="G$1" pin="SO"/>
 </segment>
@@
 <segment>
 <pinref part="U1" gate="G$1" pin="VDCDC_RF"/>
-<wire x1="86.36" y1="149.86" x2="76.2" y2="149.86" width="0.1524" layer="91"/>
-<wire x1="76.2" y1="149.86" x2="76.2" y2="139.7" width="0.1524" layer="91"/>
+<wire x1="86.36" y1="149.86" x2="63.5" y2="149.86" width="0.1524" layer="91"/>
+<wire x1="63.5" y1="149.86" x2="63.5" y2="139.7" width="0.1524" layer="91"/>
 <pinref part="U1" gate="G$1" pin="VDCDC"/>
-<wire x1="78.74" y1="139.7" x2="76.2" y2="139.7" width="0.1524" layer="91"/>
-<wire x1="76.2" y1="139.7" x2="76.2" y2="137.16" width="0.1524" layer="91"/>
-<wire x1="76.2" y1="137.16" x2="86.36" y2="137.16" width="0.1524" layer="91"/>
-<wire x1="76.2" y1="149.86" x2="58.42" y2="149.86" width="0.1524" layer="91"/>
-<junction x="76.2" y="149.86"/>
+<wire x1="73.66" y1="139.7" x2="63.5" y2="139.7" width="0.1524" layer="91"/>
+<wire x1="63.5" y1="139.7" x2="63.5" y2="137.16" width="0.1524" layer="91"/>
+<wire x1="63.5" y1="137.16" x2="86.36" y2="137.16" width="0.1524" layer="91"/>
+<wire x1="63.5" y1="149.86" x2="53.34" y2="149.86" width="0.1524" layer="91"/>
+<junction x="63.5" y="149.86"/>
 <pinref part="C3" gate="G$1" pin="1"/>
 <pinref part="L1" gate="G$1" pin="1"/>
 <pinref part="TP1" gate="G$1" pin="TP"/>
-<junction x="76.2" y="139.7"/>
-</segment>
-</net>
+<junction x="63.5" y="139.7"/>
+</segment>
+</net>

Commit message: [ FIX ] library update
Parts:
- added TP2, TP4, TP5: TESTPAD_F, mylib:TESTPAD_F
- IC1: value IC_MEMORY_8P_AT25XE011_SOP -> 1265-1137-1-ND
Changed lines of the file:
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@@
 <part name="L1" library="mylib" deviceset="INDUCTOR" device="_1608" value="2.2u"/>
 <part name="R1" library="mylib" deviceset="R_US_PAD_PAD" device="_1005"/>
-<part name="IC1" library="mylib" deviceset="IC_MEMORY_8P_*" device="_SOP" technology="AT25XE011" value="IC_MEMORY_8P_AT25XE011_SOP"/>
+<part name="IC1" library="mylib" deviceset="IC_MEMORY_8P_*" device="_SOP" technology="AT25XE011" value="1265-1137-1-ND"/>
 <part name="P+3" library="mylib" deviceset="VCC" device=""/>
 <part name="C4" library="mylib" deviceset="C_PAD_PAD_" device="1005"/>
@@
 <part name="Q2" library="mylib" deviceset="CLOCK_CRYSTAL_4" device="_2520"/>
 <part name="P+7" library="mylib" deviceset="VCC" device=""/>
+<part name="TP2" library="mylib" deviceset="TESTPAD" device="_F"/>
+<part name="TP4" library="mylib" deviceset="TESTPAD" device="_F"/>
+<part name="TP5" library="mylib" deviceset="TESTPAD" device="_F"/>
 </parts>
 <sheets>
@@
 </instance>
 <instance part="P+7" gate="VCC" x="241.3" y="114.3"/>
+<instance part="TP2" gate="1" x="17.78" y="20.32"/>
+<instance part="TP4" gate="1" x="17.78" y="17.78"/>
+<instance part="TP5" gate="1" x="17.78" y="15.24"/>
 </instances>
 <busses>
