File: DA14580_QFN40_0v5.sch (EAGLE design)
At the start: 29 parts, among them CON1 CON_TC2030-CTL-NL, IC1 IC_MEMORY_8P_AT25XE011_SOP, IC2 NC7SZ00M5XCT-ND, IC3 LDO5_3.3_SOT23, Q1 32.768k, Q2 16M/2520, U1 DA14583AT2, X1 SSW-114-02-S-S, X2 SSW-114-02-S-S

Commit message: [ 58x ] v0.5 frozen
Parts:
- added GIT1: 35b58a7, git-revision:GIT-REVISION
- added ICON1: v0.5, mylib:ICON_REVISION
Other:
- note removed: "v0.5"
- moved on the sheet: Q1, TP91, TP92, TP93
Changed lines of the file:
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@@
 <part name="TP1" library="mylib" deviceset="TESTPAD" device=""/>
 <part name="TP2" library="mylib" deviceset="TESTPAD" device=""/>
+<part name="GIT1" library="git-revision" deviceset="GIT-REVISION" device="" value="35b58a7"/>
+<part name="ICON1" library="mylib" deviceset="ICON_REVISION" device="" value="v0.5"/>
 </parts>
 <sheets>
 <sheet>
 <plain>
-<text x="162.56" y="5.08" size="12.7" layer="94">v0.5</text>
 <text x="12.7" y="167.64" size="1.778" layer="94">L1: 445-6385-1-ND</text>
-<text x="218.44" y="20.32" size="2.54" layer="94">CC-BY-SA</text>
+<text x="162.56" y="20.32" size="2.54" layer="94">CC-BY-SA</text>
+<wire x1="160.02" y1="22.86" x2="144.78" y2="22.86" width="0.1524" layer="94"/>
+<wire x1="144.78" y1="22.86" x2="144.78" y2="5.08" width="0.1524" layer="94"/>
 </plain>
 <instances>
@@
 <instance part="VDD1" gate="G$1" x="213.36" y="161.29"/>
 <instance part="P+1" gate="VCC" x="238.76" y="162.56"/>
-<instance part="Q1" gate="G$1" x="63.5" y="124.46" smashed="yes">
-<attribute name="NAME" x="60.96" y="124.46" size="1.778" layer="95" rot="R180"/>
-<attribute name="VALUE" x="66.04" y="122.682" size="1.016" layer="96"/>
-<attribute name="DIGIKEY" x="66.04" y="124.46" size="0.8128" layer="96" display="both"/>
+<instance part="Q1" gate="G$1" x="60.96" y="124.46" smashed="yes">
+<attribute name="NAME" x="58.42" y="124.46" size="1.778" layer="95" rot="R180"/>
+<attribute name="VALUE" x="63.5" y="122.682" size="1.016" layer="96"/>
+<attribute name="DIGIKEY" x="63.5" y="124.46" size="0.8128" layer="96" display="off"/>
+<attribute name="MOUSER" x="63.5" y="124.46" size="0.8128" layer="96" display="both"/>
 </instance>
 <instance part="SUPPLY7" gate="GND" x="43.18" y="127"/>
@@
 </instance>
 <instance part="L1" gate="G$1" x="73.66" y="139.7" smashed="yes">
-<attribute name="DIGIKEY" x="66.04" y="137.16" size="0.8128" layer="96" display="both"/>
+<attribute name="DIGIKEY" x="66.04" y="137.414" size="0.8128" layer="96" display="both"/>
 <attribute name="NAME" x="76.2" y="139.954" size="1.778" layer="95"/>
 <attribute name="VALUE" x="76.2" y="137.668" size="1.016" layer="96"/>
@@
 <instance part="CON1" gate="G$1" x="175.26" y="132.08"/>
 <instance part="SUPPLY5" gate="GND" x="154.94" y="127"/>
-<instance part="U$2" gate="G$1" x="205.74" y="20.32"/>
+<instance part="U$2" gate="G$1" x="248.92" y="21.59"/>
 <instance part="P+6" gate="VCC" x="152.4" y="134.62" rot="R90"/>
 <instance part="Q2" gate="G$1" x="53.34" y="132.08" smashed="yes" rot="R270">
@@
 </instance>
 <instance part="P+7" gate="VCC" x="241.3" y="114.3"/>
-<instance part="TP91" gate="1" x="17.78" y="20.32"/>
-<instance part="TP92" gate="1" x="17.78" y="17.78"/>
-<instance part="TP93" gate="1" x="17.78" y="15.24"/>
+<instance part="TP91" gate="1" x="149.86" y="12.7"/>
+<instance part="TP92" gate="1" x="149.86" y="10.16"/>
+<instance part="TP93" gate="1" x="149.86" y="7.62"/>
 <instance part="TP1" gate="1" x="63.5" y="152.4" rot="R90"/>
 <instance part="TP2" gate="1" x="53.34" y="127" rot="R270"/>
+<instance part="GIT1" gate="G$1" x="215.9" y="20.32"/>
+<instance part="ICON1" gate="G$1" x="162.56" y="5.08"/>
 </instances>
 <busses>
@@
 <segment>
 <pinref part="Q1" gate="G$1" pin="1"/>
-<wire x1="63.5" y1="127" x2="83.82" y2="127" width="0.1524" layer="91"/>
+<wire x1="60.96" y1="127" x2="83.82" y2="127" width="0.1524" layer="91"/>
 <wire x1="83.82" y1="127" x2="83.82" y2="124.46" width="0.1524" layer="91"/>
 <pinref part="U1" gate="G$1" pin="XTAL32K+"/>
@@
 <segment>
 <pinref part="U1" gate="G$1" pin="XTAL32K-"/>
-<wire x1="86.36" y1="121.92" x2="63.5" y2="121.92" width="0.1524" layer="91"/>
+<wire x1="86.36" y1="121.92" x2="60.96" y2="121.92" width="0.1524" layer="91"/>
 <pinref part="Q1" gate="G$1" pin="2"/>
 </segment>
