File: MurataBLE_FS.brd (EAGLE design)
At the start: 90 x 63 mm, 51 parts, among them CON1 WM17143CT-ND, CON2 C-2395.microSD, IC1 74LVC1G00DBV, IC2 IC_DCDC_LM27313, IC3 IC_LPC11U3XQFN33, IC4 IC_LDO_XX1117_4, IC5 IC_MEMORY_8P_AT25XE011_TSSOP, SW1 SW_TACTSW_2PP8073, SW2 SW_TACTSW_2PP8073, SW3 SW_TACTSW_2PP8073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

Commit message: update eagle version = 7.5.0; library update
Parts:
- IC4: value IC_LDO_XX1117_4 -> LDO4_3.3_SOT223
- SW1, SW2, SW3: value SW_TACTSW_2PP8073 -> (none)
- U1: value IC_BLE_LBCA2HNZYZ-711 -> LBCA2HNZYZ-711
- moved TP1 75.8 mm to (132.5, 43.9)
- moved TP2 75.8 mm to (136.0, 43.9)
- moved C6 8.59 mm to (61.6, 18.6), turned to 90 degrees
- moved R2 8.04 mm to (55.5, 24.2), turned to 180 degrees
- moved R3 6.96 mm to (60.2, 18.6), turned to 270 degrees
- moved C5 6.40 mm to (63.2, 18.6), turned to 90 degrees
- moved D1 5.41 mm to (56.2, 17.4), turned to 180 degrees
- moved R4 5.39 mm to (58.5, 20.4), turned to 270 degrees
- moved L1 2.73 mm to (52.7, 21.5), turned to 270 degrees
- moved IC2 1.70 mm to (55.7, 21.1), turned to 0 degrees
Connections:
- net N$7: now also IC2.1; no longer IC2.5
- net VIN: now also IC2.5; no longer IC2.1
Routing:
- net VPP: track 38.1 -> 16.4 mm
- net N$8: track 12.6 -> 1.60 mm, vias 2 -> 0
- net GND: track 19.2 -> 9.49 mm, vias 69 -> 66
- net N$7: track 5.20 -> 4.54 mm
