File: DA14580_QFN40.sch (EAGLE design)
At the start: 31 parts, among them CON1 CON_TC2030-CTL-NL, IC1 IC_MEMORY_8P_AT25XE011_SOP, IC2 NC7SZ00M5XCT-ND, IC3 LDO5_3.3_SOT23, Q1 32.768k, Q2 16M/2520, U1 DA14583AT2, X1 SSW-114-02-S-S, X2 SSW-114-02-S-S

Commit message: [ 58x ] font alignment
Parts:
- GIT1: value (none) -> b61e68f
- ICON1: device mylib:ICON_REVISION -> mylib:ICON_REVISION_1.2
- TP3: value TPPAD1-13 -> (none); device testpad_local:TPPAD1-13 -> mylib:TESTPAD_4020
Connections:
- net GND: now also TP3.1; no longer TP3.TP
Other:
- moved on the sheet: TP91, TP92, TP93
Changed lines of the file:
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@@
 <part name="IC3" library="mylib" deviceset="LDO5_*" device="_SOT23" technology="3.3" value="LDO5_3.3_SOT23"/>
 <part name="IC2" library="74xx-little-us_local" deviceset="74*1G00" device="DBV" technology="LVC" value="NC7SZ00M5XCT-ND"/>
-<part name="TP3" library="testpad_local" deviceset="TP" device="PAD1-13"/>
 <part name="C6" library="mylib" deviceset="C_SMD_*" device="_1005" technology="10P" value="NM"/>
 <part name="C7" library="mylib" deviceset="C_SMD_*" device="_1005" value="NM"/>
@@
 <part name="TP1" library="mylib" deviceset="TESTPAD" device=""/>
 <part name="TP2" library="mylib" deviceset="TESTPAD" device=""/>
-<part name="GIT1" library="git-revision" deviceset="GIT-REVISION" device=""/>
-<part name="ICON1" library="mylib" deviceset="ICON_REVISION" device="" value="v0.6"/>
+<part name="GIT1" library="git-revision" deviceset="GIT-REVISION" device="" value="b61e68f"/>
+<part name="ICON1" library="mylib" deviceset="ICON_REVISION" device="_1.2" value="v0.6"/>
+<part name="TP3" library="mylib" deviceset="TESTPAD" device="_4020"/>
 </parts>
 <sheets>
@@
 <text x="12.7" y="167.64" size="1.778" layer="94">L1: 445-6385-1-ND</text>
 <text x="162.56" y="20.32" size="2.54" layer="94">CC-BY-SA</text>
+<wire x1="160.02" y1="22.86" x2="144.78" y2="22.86" width="0.1524" layer="94"/>
+<wire x1="144.78" y1="22.86" x2="144.78" y2="5.08" width="0.1524" layer="94"/>
 </plain>
 <instances>
@@
 <instance part="IC2" gate="A" x="228.6" y="54.61"/>
 <instance part="IC2" gate="P" x="217.17" y="72.39"/>
-<instance part="TP3" gate="G$1" x="210.82" y="40.64"/>
 <instance part="C6" gate="G$1" x="134.62" y="160.02" rot="R90"/>
 <instance part="C7" gate="G$1" x="139.7" y="157.48"/>
@@
 </instance>
 <instance part="P+7" gate="VCC" x="241.3" y="114.3"/>
-<instance part="TP91" gate="1" x="17.78" y="20.32"/>
-<instance part="TP92" gate="1" x="17.78" y="17.78"/>
-<instance part="TP93" gate="1" x="17.78" y="15.24"/>
+<instance part="TP91" gate="1" x="149.86" y="15.24"/>
+<instance part="TP92" gate="1" x="149.86" y="12.7"/>
+<instance part="TP93" gate="1" x="149.86" y="10.16"/>
 <instance part="TP1" gate="1" x="63.5" y="152.4" rot="R90"/>
 <instance part="TP2" gate="1" x="53.34" y="127" rot="R270"/>
 <instance part="GIT1" gate="G$1" x="215.9" y="20.32"/>
 <instance part="ICON1" gate="G$1" x="162.56" y="5.08"/>
+<instance part="TP3" gate="1" x="213.36" y="38.1">
+<attribute name="DIGIKEY" x="213.36" y="35.56" size="0.8128" layer="96" display="both"/>
+</instance>
 </instances>
 <busses>
@@
 <segment>
 <pinref part="SUPPLY4" gate="GND" pin="GND"/>
-<pinref part="TP3" gate="G$1" pin="TP"/>
 <wire x1="210.82" y1="38.1" x2="210.82" y2="35.56" width="0.1524" layer="91"/>
+<pinref part="TP3" gate="1" pin="1"/>
 </segment>
 <segment>

Commit message: replace IC2/3 to smaller outlined devices
Parts:
- added P1, P2: (no value), mylib:PCB_CORNER_NH
- added P3, P4: (no value), mylib:PCB_CORNER
- IC2: value NC7SZ00M5XCT-ND -> (none); device 74xx-little-us_local:74LVC1G00DBV -> mylib:74LVC1G00_DRL
- IC3: value LDO5_3.3_SOT23 -> (none); device mylib:LDO5_3.3_SOT23 -> mylib:LDO4_3.3_SC82-AB
Connections:
- net !RESET!: now also IC2.1A, IC2.1B; no longer IC2A.I0, IC2A.I1
- net GND: now also IC2.GND; no longer IC2P.GND
- net RESET: now also IC2.1Y; no longer IC2A.O
- net VCC: now also IC2.VCC; no longer IC2P.VCC
- net VDD: now also IC3.OUT/EN/NC; no longer IC3.E
Other:
- moved on the sheet: C2, C5, R1
